File: pellet_burner.kicad_pcb (KiCad board)
At the start: 4 copper layers, 100 x 80 mm, 170 parts, among them J6 Power input, J7 USB4110-GF-A, Q1 IRLML6344TRPBF, Q2 IRLML6344TRPBF, Q3 IRLML6344TRPBF, Q4 IRLML6344TRPBF, Q5 IRLML6344TRPBF, Q6 IRLML6344TRPBF, Q7 IRLML6344TRPBF, Q8 IRLML6344TRPBF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

Commit message: up
Parts:
- added J13: 5v, TerminalBlock:TerminalBlock_MaiXu_MX126-5.0-02P_1x02_P5.00mm, F.Cu at (54.6, 122.7)
- J6: value Power input -> 24V Power input
- moved SW2 5.23 mm to (110.4, 76.2), turned to 0 degrees
Connections:
- net /EN renamed Net-(U3-EN)
- net D+ renamed Net-(U3-GPIO20/U1CTS/ADC2_CH9/CLK_OUT1/USB_D+)
- net D- renamed Net-(U3-GPIO19/U1RTS/ADC2_CH8/CLK_OUT2/USB_D-)
- net GPIO1 renamed Net-(U3-GPIO1/TOUCH1/ADC1_CH0)
- net GPIO2 renamed Net-(U3-GPIO2/TOUCH2/ADC1_CH1)
- net GPIO45 renamed Net-(U3-GPIO45)
- net GPIO46 renamed Net-(U3-GPIO46)
- net RX/GPIO44 renamed Net-(U3-U0RXD/GPIO44/CLK_OUT2)
- net TX/GPIO43 renamed Net-(U3-U0TXD/GPIO43/CLK_OUT1)
- J6 pad 1: GND -> +24V
- J6 pad 2: +24V -> GND
- R34 pad 2: BOOT -> Net-(U3-GPIO0/BOOT)
- SW2 pad 1: GND -> Net-(U3-GPIO0/BOOT)
- SW2 pad 2: BOOT -> GND
- U3 pad 27: BOOT -> Net-(U3-GPIO0/BOOT)
Routing:
- net +5V: track 185.8 -> 198.7 mm
- net Net-(U3-GPIO0/BOOT): track 0.00 -> 10.0 mm
- net BOOT: track 10.0 -> 0.00 mm
- net GND: track 184.7 -> 188.2 mm, vias 38 -> 46
- net +24V: track 58.9 -> 61.9 mm
- net (no net): vias 0 -> 1
- added copper zone on B.Cu, net GND
- added copper zone on F.Cu, net GND
