File: pellet_burner.kicad_sch (KiCad schematic)
At the start: 166 parts, among them J6 Power input, J7 USB4110-GF-A, Q1 IRLML6344TRPBF, Q2 IRLML6344TRPBF, Q3 IRLML6344TRPBF, Q4 IRLML6344TRPBF, Q5 IRLML6344TRPBF, Q6 IRLML6344TRPBF, Q7 IRLML6344TRPBF, Q8 IRLML6344TRPBF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

Commit message: up
Parts:
- added J13: 5v, TerminalBlock:TerminalBlock_MaiXu_MX126-5.0-02P_1x02_P5.00mm, symbol Connector:Conn_01x02_Pin
- J6: value Power input -> 24V Power input
Connections:
- net +24V: now also J6.1 (Pin_1); no longer J6.2 (Pin_2)
- net +5V: now also J13.1 (Pin_1)
- net GND: now also J6.2 (Pin_2), SW2.2, J13.2 (Pin_2); no longer J6.1 (Pin_1), SW2.1
- net BOOT: no longer names the net of R34.2, U3.27 (GPIO0/BOOT)
- net BOOT: now also SW2.1; no longer SW2.2
- net D+: no longer names the net of J7.A6, J7.B6, U3.14 (GPIO20/U1CTS/ADC2_CH9/CLK_OUT1/USB_D+)
- net D-: no longer names the net of J7.A7, J7.B7, U3.13 (GPIO19/U1RTS/ADC2_CH8/CLK_OUT2/USB_D-)
- net EN: no longer names the net of C15.1, R3.2, SW1.2, U3.3 (EN)
- net GPIO1: no longer names the net of J18.2, R36.2, R38.2, U3.39 (GPIO1/TOUCH1/ADC1_CH0)
- net GPIO2: no longer names the net of J15.2, R35.2, R37.2, U3.38 (GPIO2/TOUCH2/ADC1_CH1)
- net GPIO45: no longer names the net of R12.1, U3.26 (GPIO45)
- net GPIO46: no longer names the net of R11.1, U3.16 (GPIO46)
- net RX/GPIO44: no longer names the net of J1.3, U3.36 (U0RXD/GPIO44/CLK_OUT2)
- net TX/GPIO43: no longer names the net of J1.2, U3.37 (U0TXD/GPIO43/CLK_OUT1)
Other:
- note added: "Power"
- note added: "USB-C port"
- note removed: "24V Input"
- note removed: "BOOT pin"
- note removed: "Buck converter 5 VDC - VOUT 3.3 VDC"
- note removed: "Buck converter VIN 3.8...32VDC - VOUT 5 VDC"
- note removed: "Enable pin"
- note removed: "UART0"
- note removed: "USB"
- moved on the sheet: C1, C10, C11, C12, C13, C14, C15, C16, C17, C18, C19, C2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
